File: hands.kicad_pcb (KiCad board)
At the start: 2 copper layers, 289.8 x 99.8 mm, 78 parts, among them SW1 SW_Push, SW10 SW_Push, SW11 SW_Push, SW12 SW_Push, SW13 SW_Push, SW14 SW_Push, SW15 SW_Push, SW16 SW_Push, SW17 SW_Push, SW18 SW_Push, SW19 SW_Push, SW2 SW_Push, SW20 SW_Push, SW21 SW_Push, SW22 SW_Push, SW23 SW_Push, SW24 SW_Push, SW25 SW_Push, SW26 SW_Push, SW27 SW_Push, SW28 SW_Push, SW29 SW_Push, SW3 SW_Push, SW30 SW_Push, SW31 SW_Push, SW32 SW_Push, SW33 SW_Push, SW34 SW_Push, SW35 SW_Push, SW36 SW_Push, SW4 SW_Push, SW5 SW_Push, SW6 SW_Push, SW7 SW_Push, SW8 SW_Push, SW9 SW_Push, U1 XIAO-RP2040-DIP

Commit message: Fixed key pitch and added mounting hole
Parts:
- added M2: MountingHole_2.2mm_M2, MountingHole:MountingHole_2.2mm_M2, F.Cu at (87.9, 125.9)
- added M2: MountingHole_2.2mm_M2, MountingHole:MountingHole_2.2mm_M2, F.Cu at (254.1, 125.9)
- added M2: MountingHole_2.2mm_M2, MountingHole:MountingHole_2.2mm_M2, F.Cu at (26.1, 49.9)
- added M2: MountingHole_2.2mm_M2, MountingHole:MountingHole_2.2mm_M2, F.Cu at (154.4, 83.1)
- added M2: MountingHole_2.2mm_M2, MountingHole:MountingHole_2.2mm_M2, F.Cu at (125.9, 83.1)
- added M2: MountingHole_2.2mm_M2, MountingHole:MountingHole_2.2mm_M2, F.Cu at (140.1, 72.4)
- added M2: MountingHole_2.2mm_M2, MountingHole:MountingHole_2.2mm_M2, F.Cu at (254.1, 49.9)
- added M2: MountingHole_2.2mm_M2, MountingHole:MountingHole_2.2mm_M2, F.Cu at (192.4, 125.9)
- added M2: MountingHole_2.2mm_M2, MountingHole:MountingHole_2.2mm_M2, F.Cu at (26.1, 125.9)
- moved D31 53.9 mm to (244.6, 100.9)
- moved SW28 53.1 mm to (244.6, 97.4)
- moved D21 52.9 mm to (244.6, 81.9)
- moved SW19 52.5 mm to (244.6, 78.4)
- moved D1 52.4 mm to (244.6, 51.1)
- moved D11 52.4 mm to (244.6, 62.9)
- moved SW10 52.2 mm to (244.6, 59.4)
- moved D32 49.3 mm to (225.6, 100.9)
- moved SW29 48.4 mm to (225.6, 97.4)
- moved D22 48.2 mm to (225.6, 81.9)
- moved SW20 47.7 mm to (225.6, 78.4)
- moved D12 47.6 mm to (225.6, 67.7)
- moved D2 47.6 mm to (225.6, 62.9)
- moved SW1 47.5 mm to (225.6, 59.4)
- moved D33 44.7 mm to (206.6, 100.9)
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Routing:
- net Net-(D23-K): track 338.7 -> 242.5 mm
- net Net-(D12-K): track 332.1 -> 238.7 mm
- net Net-(D1-K): track 336.8 -> 248.0 mm, vias 10 -> 0
- net Net-(D34-K): track 241.5 -> 186.9 mm
- net /PIN1: track 194.7 -> 150.4 mm
- net /PIN3: track 168.4 -> 129.2 mm
- net /PIN8: track 173.3 -> 134.2 mm
- net /PIN10: track 178.7 -> 141.5 mm
- net /PIN4: track 151.1 -> 116.8 mm
- net /PIN7: track 153.3 -> 119.7 mm
- net /PIN2: track 148.9 -> 117.5 mm
- net /PIN9: track 153.9 -> 122.5 mm
- net /PIN6: track 99.6 -> 75.9 mm
- net /PIN5: track 117.2 -> 97.5 mm
- net Net-(D41-K): track 50.7 -> 39.2 mm
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Other:
- board size 289.8 x 99.8 mm -> 237.5 x 85.5 mm
